File: distress_monitor_board/distress_monitor_board.kicad_sch (KiCad schematic)
At the start: 11 parts

Commit message: Kicad schematic finished
Parts:
- added J1: Barrel_Jack, symbol Connector:Barrel_Jack
- added J2: USB_B_Micro, symbol Connector:USB_B_Micro
- gave numbers to parts that had none: 10
Connections:
- net Feather_RST: no longer R2.2, SW2.1
- net GND: now also J1.2, J2.5 (GND)
- net VCC: now also J1.1, J2.1 (VBUS)
- new net PUSH_BUTTON_PIN: R2.2, SW2.1, U?. (USB)

Commit message: minor change to schematic
Parts:
- gave numbers to parts that had none: 1
- renumbered U1 to U2, U2 to U3, U3 to U4, U4 to U5, U5 to U6
Changed lines of the file:
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@@
   (symbol (lib_id "distress_monitor_library:Neo-6m") (at 49.53 175.26 270) (unit 1)
     (in_bom yes) (on_board yes) (fields_autoplaced)
-    (property "Reference" "U5" (id 0) (at 48.26 165.1 90))
+    (property "Reference" "U6" (id 0) (at 48.26 165.1 90))
     (property "Value" "Neo-6m" (id 1) (at 48.26 167.64 90))
     (property "Footprint" "" (id 2) (at 49.53 175.26 0)
@@
   (symbol (lib_id "distress_monitor_library:Feather_esp32") (at 152.4 91.44 0) (unit 1)
     (in_bom yes) (on_board yes) (fields_autoplaced)
-    (property "Reference" "U?" (id 0) (at 152.4 67.31 0))
+    (property "Reference" "U1" (id 0) (at 152.4 67.31 0))
     (property "Value" "Feather_esp32" (id 1) (at 152.4 69.85 0))
     (property "Footprint" "" (id 2) (at 149.86 91.44 0)
@@
   (symbol (lib_id "distress_monitor_library:ADXL345") (at 45.72 71.12 270) (unit 1)
     (in_bom yes) (on_board yes) (fields_autoplaced)
-    (property "Reference" "U2" (id 0) (at 45.085 54.61 90))
+    (property "Reference" "U3" (id 0) (at 45.085 54.61 90))
     (property "Value" "ADXL345" (id 1) (at 45.085 57.15 90))
     (property "Footprint" "" (id 2) (at 45.72 71.12 0)
@@
   (symbol (lib_id "distress_monitor_library:ST7735_TFT_LCD_1.8") (at 36.83 111.76 180) (unit 1)
     (in_bom yes) (on_board yes) (fields_autoplaced)
-    (property "Reference" "U3" (id 0) (at 36.83 95.25 0))
+    (property "Reference" "U4" (id 0) (at 36.83 95.25 0))
     (property "Value" "ST7735_TFT_LCD_1.8" (id 1) (at 36.83 97.79 0))
     (property "Footprint" "" (id 2) (at 45.72 110.49 0)
@@
   (symbol (lib_id "distress_monitor_library:D24V10F3") (at 44.45 27.94 270) (unit 1)
     (in_bom yes) (on_board yes) (fields_autoplaced)
-    (property "Reference" "U1" (id 0) (at 45.085 15.24 90))
+    (property "Reference" "U2" (id 0) (at 45.085 15.24 90))
     (property "Value" "D24V10F3" (id 1) (at 45.085 17.78 90))
     (property "Footprint" "" (id 2) (at 44.45 27.94 0)
@@
   (symbol (lib_id "distress_monitor_library:HR_sensor") (at 45.72 148.59 270) (unit 1)
     (in_bom yes) (on_board yes) (fields_autoplaced)
-    (property "Reference" "U4" (id 0) (at 47.625 139.7 90))
+    (property "Reference" "U5" (id 0) (at 47.625 139.7 90))
     (property "Value" "HR_sensor" (id 1) (at 47.625 142.24 90))
     (property "Footprint" "" (id 2) (at 45.72 148.59 0)
@@
       (reference "SW2") (unit 1) (value "Distress_Button") (footprint "")
     )
+    (path "/2ad1f6ee-a15f-4b51-adc8-ba2d9ec37739"
+      (reference "U1") (unit 1) (value "Feather_esp32") (footprint "")
+    )
     (path "/8e698cac-c90c-4684-8518-14b3d0d15feb"
-      (reference "U1") (unit 1) (value "D24V10F3") (footprint "")
+      (reference "U2") (unit 1) (value "D24V10F3") (footprint "")
     )
     (path "/343f3478-d3c8-4d3a-954a-45ebe01f8afa"
-      (reference "U2") (unit 1) (value "ADXL345") (footprint "")
+      (reference "U3") (unit 1) (value "ADXL345") (footprint "")
     )
     (path "/4f1b5351-68e5-459a-a096-42909c5810e0"
-      (reference "U3") (unit 1) (value "ST7735_TFT_LCD_1.8") (footprint "")
+      (reference "U4") (unit 1) (value "ST7735_TFT_LCD_1.8") (footprint "")
     )
     (path "/f076b1f9-5e56-4803-bdb6-bc8c9bc5a8b8"
-      (reference "U4") (unit 1) (value "HR_sensor") (footprint "")
+      (reference "U5") (unit 1) (value "HR_sensor") (footprint "")
     )
     (path "/1784dfaf-d018-4971-b08e-afdc12a4a1ba"
-      (reference "U5") (unit 1) (value "Neo-6m") (footprint "")
-    )
-    (path "/2ad1f6ee-a15f-4b51-adc8-ba2d9ec37739"
-      (reference "U?") (unit 1) (value "Feather_esp32") (footprint "")
+      (reference "U6") (unit 1) (value "Neo-6m") (footprint "")
     )
     (path "/3a28bbed-aab5-49ef-856d-35d3415811a1"
